File: pcb board/gsm_LoRa/gsm_LoRa_due.sch (EAGLE design)
At the start: 36 parts, among them IC1 TPS22810TDBVRQ1, IC3 DS3231MZ+, X1 22-23-2021

Commit message: added SPI connector
Parts:
- added SPI: JST-XH-06-PIN-ROUND-PAD, Rembrandt Electronics - JST XH Connectors v1-0:JST-XH-06-PIN-ROUND-PAD
Connections:
- new net CS: SPI-4.S, U$1.A3
- new net MISO: SPI-1.S, U$1.MISO
- new net MOSI: SPI-2.S, U$1.MOSI
- new net SCK: SPI-3.S, U$1.SCK
- net +3V3: now also SPI-5.S
- net 12VIN: now also U$10.+IN, U$10.+IN1; no longer U$10.-IN, U$10.-IN1
- net DC-DC: now also U$10.+OUT, U$10.+OUT1; no longer U$10.-OUT, U$10.-OUT1
- net GND: now also SPI-6.S, U$10.-IN, U$10.-IN1, U$10.-OUT, U$10.-OUT1; no longer U$10.+IN, U$10.+IN1, U$10.+OUT, U$10.+OUT1
Other:
- moved on the sheet: C3, C4, R5, R6, S1

Commit message: Updated names on traces
Parts:
- renumbered BATT to BATTERY
Changed lines of the file:
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@@
 <part name="POWER" library="con-molex" library_urn="urn:adsk.eagle:library:165" deviceset="22-23-2021" device=""/>
 <part name="TRIGGER" library="con-molex" library_urn="urn:adsk.eagle:library:165" deviceset="22-23-2021" device=""/>
-<part name="BATT" library="con-molex" library_urn="urn:adsk.eagle:library:165" deviceset="22-23-2021" device=""/>
+<part name="BATTERY" library="con-molex" library_urn="urn:adsk.eagle:library:165" deviceset="22-23-2021" device=""/>
 <part name="C8" library="eagle-ltspice" library_urn="urn:adsk.eagle:library:217" deviceset="C" device="C0603" package3d_urn="urn:adsk.eagle:package:13262/1"/>
 <part name="U$12" library="microbuilder" deviceset="GND" device=""/>
@@
 <attribute name="NAME" x="121.92" y="35.778" size="1.524" layer="95"/>
 </instance>
-<instance part="BATT" gate="-1" x="36.62" y="205.42" smashed="yes" rot="R180">
+<instance part="BATTERY" gate="-1" x="36.62" y="205.42" smashed="yes" rot="R180">
 <attribute name="NAME" x="34.08" y="206.182" size="1.524" layer="95" rot="R180"/>
 <attribute name="VALUE" x="37.382" y="204.023" size="1.778" layer="96" rot="R180"/>
 </instance>
-<instance part="BATT" gate="-2" x="36.62" y="207.96" smashed="yes" rot="R180">
+<instance part="BATTERY" gate="-2" x="36.62" y="207.96" smashed="yes" rot="R180">
 <attribute name="NAME" x="34.08" y="208.722" size="1.524" layer="95" rot="R180"/>
 </instance>
@@
 </segment>
 <segment>
-<pinref part="BATT" gate="-1" pin="S"/>
+<pinref part="BATTERY" gate="-1" pin="S"/>
 <wire x1="39.16" y1="205.42" x2="44" y2="205.42" width="0.1524" layer="91"/>
 <wire x1="44" y1="205.42" x2="44" y2="205.5" width="0.1524" layer="91"/>
@@
 <segment>
 <pinref part="U$11" gate="G$1" pin="BATT"/>
-<pinref part="BATT" gate="-2" pin="S"/>
+<pinref part="BATTERY" gate="-2" pin="S"/>
 <wire x1="57.8" y1="208.38" x2="39.16" y2="208.38" width="0.1524" layer="91"/>
 <wire x1="39.16" y1="208.38" x2="39.16" y2="207.96" width="0.1524" layer="91"/>

Commit message: Added power IC switch for GSM Updated names of components
Parts:
- added C10, C9: (no value), eagle-ltspice:CC0603
- added GSM-PWR: 0R-JUMPB, jump-0r-smd:0R-JUMPB
- added IC2: TPS22810TDBVRQ1, TPS22810TDBVRQ1:TPS22810TDBVRQ1
Connections:
- new net GSMPWR: C10.1, IC2.VOUT, U$9.VCC
- new net GSMSW: GSM-PWR-0R.2, IC2.EN/UVLO
- new net GSM_PSW: GSM-PWR-0R.3, U$1.A2
- net 4V4: now also C9.2, GSM-PWR-0R.1, IC2.VIN; no longer U$9.VCC
- net GND: now also C10.2, C9.1, IC2.GND
Changed lines of the file:
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@@
 <part name="X1" library="con-molex" library_urn="urn:adsk.eagle:library:165" deviceset="22-23-2021" device=""/>
 <part name="SPI" library="Rembrandt Electronics - JST XH Connectors v1-0" deviceset="JST-XH-06-PIN" device="-ROUND-PAD"/>
+<part name="IC2" library="TPS22810TDBVRQ1" deviceset="TPS22810TDBVRQ1" device=""/>
+<part name="C9" library="eagle-ltspice" library_urn="urn:adsk.eagle:library:217" deviceset="C" device="C0603" package3d_urn="urn:adsk.eagle:package:13262/1"/>
+<part name="C10" library="eagle-ltspice" library_urn="urn:adsk.eagle:library:217" deviceset="C" device="C0603" package3d_urn="urn:adsk.eagle:package:13262/1"/>
+<part name="U$14" library="microbuilder" deviceset="GND" device=""/>
+<part name="U$15" library="microbuilder" deviceset="GND" device=""/>
+<part name="U$16" library="microbuilder" deviceset="GND" device=""/>
+<part name="GSM-PWR" library="jump-0r-smd" library_urn="urn:adsk.eagle:library:251" deviceset="0R-JUMP" device="B" package3d_urn="urn:adsk.eagle:package:15387/1"/>
 </parts>
 <sheets>
@@
 <attribute name="NAME" x="-81.28" y="219.202" size="1.524" layer="95" rot="R180"/>
 </instance>
+<instance part="IC2" gate="G$1" x="-149.2" y="145.32" smashed="yes">
+<attribute name="NAME" x="-119.99" y="152.94" size="1.778" layer="95" align="center-left"/>
+<attribute name="VALUE" x="-119.99" y="150.4" size="1.778" layer="96" align="center-left"/>
+</instance>
+<instance part="C9" gate="G$1" x="-160.3" y="138.08" smashed="yes" rot="R180">
+<attribute name="NAME" x="-161.824" y="137.699" size="1.778" layer="95" rot="R180"/>
+<attribute name="VALUE" x="-161.824" y="142.779" size="1.778" layer="96" rot="R180"/>
+</instance>
+<instance part="C10" gate="G$1" x="-109.3" y="140.58" smashed="yes">
+<attribute name="NAME" x="-107.776" y="140.961" size="1.778" layer="95"/>
+<attribute name="VALUE" x="-107.776" y="135.881" size="1.778" layer="96"/>
+</instance>
+<instance part="U$14" gate="G$1" x="-109.41" y="131.76" smashed="yes">
+<attribute name="VALUE" x="-110.934" y="129.22" size="1.27" layer="96"/>
+</instance>
+<instance part="U$15" gate="G$1" x="-160.21" y="130.26" smashed="yes">
+<attribute name="VALUE" x="-161.734" y="127.72" size="1.27" layer="96"/>
+</instance>
+<instance part="U$16" gate="G$1" x="-154.91" y="128.26" smashed="yes">
+<attribute name="VALUE" x="-156.434" y="125.72" size="1.27" layer="96"/>
+</instance>
+<instance part="GSM-PWR" gate="-0R" x="-142.24" y="119.38" smashed="yes">
+<attribute name="NAME" x="-139.7" y="123.19" size="1.778" layer="95"/>
+</instance>
+<instance part="GSM-PWR" gate="G$2" x="-144.78" y="121.92" smashed="yes"/>
 </instances>
 <busses>
@@
 <label x="-71.12" y="218.44" size="1.778" layer="95"/>
 </segment>
+<segment>
+<pinref part="IC2" gate="G$1" pin="GND"/>
+<pinref part="U$16" gate="G$1" pin="GND"/>
+<wire x1="-149.2" y1="142.78" x2="-154.91" y2="142.78" width="0.1524" layer="91"/>
+<wire x1="-154.91" y1="142.78" x2="-154.91" y2="130.8" width="0.1524" layer="91"/>
+</segment>
+<segment>
+<pinref part="C10" gate="G$1" pin="2"/>
+<pinref part="U$14" gate="G$1" pin="GND"/>
+<wire x1="-109.3" y1="135.5" x2="-109.41" y2="135.5" width="0.1524" layer="91"/>
+<wire x1="-109.41" y1="135.5" x2="-109.41" y2="134.3" width="0.1524" layer="91"/>
+</segment>
+<segment>
+<pinref part="C9" gate="G$1" pin="1"/>
+<pinref part="U$15" gate="G$1" pin="GND"/>
+<wire x1="-160.3" y1="135.54" x2="-160.3" y2="132.8" width="0.1524" layer="91"/>
+<wire x1="-160.3" y1="132.8" x2="-160.21" y2="132.8" width="0.1524" layer="91"/>
+</segment>
 </net>
 <net name="+3V3" class="0">
@@
 <wire x1="224.5" y1="125.56" x2="224.5" y2="125.5" width="0.1524" layer="91"/>
 <label x="222" y="125.5" size="1.778" layer="95"/>
+</segment>
+<segment>
+<pinref part="S1" gate="1" pin="P"/>
+<wire x1="66.84" y1="140.42" x2="66.84" y2="140.46" width="0.1524" layer="91"/>
+<wire x1="66.84" y1="140.46" x2="58.42" y2="140.46" width="0.1524" layer="91"/>
+<label x="58.42" y="140.46" size="1.778" layer="95"/>
+</segment>
+<segment>
+<pinref part="C9" gate="G$1" pin="2"/>
+<wire x1="-160.3" y1="143.16" x2="-160.3" y2="145.64" width="0.1524" layer="91"/>
+<pinref part="IC2" gate="G$1" pin="VIN"/>
+<wire x1="-160.3" y1="145.64" x2="-149.2" y2="145.64" width="0.1524" layer="91"/>
+<wire x1="-149.2" y1="145.64" x2="-149.2" y2="145.32" width="0.1524" layer="91"/>
+<label x="-160.16" y="145.54" size="1.778" layer="95"/>
+</segment>
+<segment>
+<pinref part="GSM-PWR" gate="-0R" pin="1"/>
+<wire x1="-142.24" y1="121.92" x2="-142.24" y2="127" width="0.1524" layer="91"/>
+<label x="-142.24" y="127" size="1.778" layer="95"/>
 </segment>
 <segment>
@@
 <label x="-85" y="155.5" size="1.778" layer="95"/>
 </segment>
-<segment>
-<pinref part="U$9" gate="G$1" pin="VCC"/>
-<wire x1="-7.7" y1="147.7" x2="-19" y2="147.7" width="0.1524" layer="91"/>
-<wire x1="-19" y1="147.7" x2="-19" y2="148" width="0.1524" layer="91"/>
-<label x="-19" y="148" size="1.778" layer="95"/>
-</segment>
-<segment>
-<pinref part="S1" gate="1" pin="P"/>
-<wire x1="66.84" y1="140.42" x2="66.84" y2="140.46" width="0.1524" layer="91"/>
-<wire x1="66.84" y1="140.46" x2="58.42" y2="140.46" width="0.1524" layer="91"/>
-<label x="58.42" y="140.46" size="1.778" layer="95"/>
-</segment>
 </net>
 <net name="TXD_GSM" class="0">
@@
 </segment>
 </net>
+<net name="GSMPWR" class="0">
+<segment>
+<pinref part="C10" gate="G$1" pin="1"/>
+<wire x1="-109.3" y1="145.32" x2="-109.3" y2="143.12" width="0.1524" layer="91"/>
+<pinref part="IC2" gate="G$1" pin="VOUT"/>
+<wire x1="-116.18" y1="145.32" x2="-109.3" y2="145.32" width="0.1524" layer="91"/>
+<label x="-109.22" y="144.78" size="1.778" layer="95"/>
+</segment>
+<segment>
+<pinref part="U$9" gate="G$1" pin="VCC"/>
+<wire x1="-7.7" y1="147.7" x2="-19" y2="147.7" width="0.1524" layer="91"/>
+<wire x1="-19" y1="147.7" x2="-19" y2="148" width="0.1524" layer="91"/>
+<label x="-19" y="148" size="1.778" layer="95"/>
+</segment>
+</net>
+<net name="GSMSW" class="0">
+<segment>
+<pinref part="IC2" gate="G$1" pin="EN/UVLO"/>
+<wire x1="-149.2" y1="140.24" x2="-149.2" y2="140.08" width="0.1524" layer="91"/>
+<wire x1="-149.2" y1="140.08" x2="-152.3" y2="140.08" width="0.1524" layer="91"/>
+<wire x1="-152.3" y1="140.08" x2="-152.3" y2="134.08" width="0.1524" layer="91"/>
+<wire x1="-152.3" y1="134.08" x2="-147.3" y2="134.08" width="0.1524" layer="91"/>
+<label x="-150.3" y="134.08" size="1.778" layer="95"/>
+</segment>
+<segment>
+<pinref part="GSM-PWR" gate="-0R" pin="2"/>
+<wire x1="-139.7" y1="119.38" x2="-134.62" y2="119.38" width="0.1524" layer="91"/>
+<label x="-134.62" y="119.38" size="1.778" layer="95"/>
+</segment>
+</net>
+<net name="GSM_PSW" class="0">
+<segment>
+<pinref part="U$1" gate="G$1" pin="A2"/>
+<wire x1="157.6" y1="115.38" x2="147.32" y2="115.38" width="0.1524" layer="91"/>
+<wire x1="147.32" y1="115.38" x2="147.32" y2="116.84" width="0.1524" layer="91"/>
+<label x="147.32" y="116.84" size="1.778" layer="95"/>
+</segment>
+<segment>
+<pinref part="GSM-PWR" gate="-0R" pin="3"/>
+<wire x1="-142.24" y1="116.84" x2="-142.24" y2="111.76" width="0.1524" layer="91"/>
+<label x="-142.24" y="111.76" size="1.778" layer="95"/>
+</segment>
+</net>

Commit message: addded ring pin to A0
Parts:
- C1, C10, C2, C3, C8, C9: value (none) -> 1uF
- C4: value (none) -> 100nF
Connections:
- removed net RTCVIN: U$1.A0
- new net RING: U$1.A0, U$9.RING
Other:
- note added: "Adafruit Feather M0 RFM96"
- note added: "CONNECTORS"
- note added: "CUSTOM DUE TRIGGER SWITCH"
- note added: "GSM SWITCH and POWER SUPPLY"
- note added: "LI-ION BATTERY CHARGER"
- note added: "REAL TIME CLOCK"
- moved on the sheet: BATTERY-1, BATTERY-2, C1, C10, C14, C2, C3, C4, C5, C6, C7, C8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
