File: pcb board/atsamdg21/atsamdg21_v1.20.sch (EAGLE design)
At the start: 54 parts, among them IC1 DS3231MZ+, IC2 TPS22810TDBVRQ1, SW1 SPST_TACT-KMR2, U1 ATSAMD21G18A-AU, U2 AP2112K-3.3, U4 RFM69HCW, X1 TSW-105-07-G-S, X2 32.768, X3 microUSB, X4 uFL, X6 TSW-103-08-G-S

Commit message: 05/22 update
Connections:
- removed net N$3: R3.2, U1.!RESETN
- removed net N$8: C17.1
- net !RESET: now also R3.2, U1.!RESETN
- net N$6: now also C17.1
Changed lines of the file:
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@@
 <?xml version="1.0" encoding="utf-8"?>
 <!DOCTYPE eagle SYSTEM "eagle.dtd">
-<eagle version="9.5.1">
+<eagle version="9.6.1">
 <drawing>
 <settings>
-<setting alwaysvectorfont="yes"/>
+<setting alwaysvectorfont="no"/>
 <setting verticaltext="up"/>
 </settings>
@@
 </segment>
 </net>
-<net name="N$3" class="0">
-<segment>
-<pinref part="U1" gate="G$1" pin="!RESETN"/>
-<wire x1="50.324" y1="227.076" x2="44.704" y2="227.076" width="0.1524" layer="91"/>
-<pinref part="R3" gate="G$1" pin="2"/>
-<wire x1="44.704" y1="227.076" x2="44.704" y2="228.156" width="0.1524" layer="91"/>
-</segment>
-</net>
 <net name="N$1" class="0">
 <segment>
@@
 <pinref part="SW1" gate="G$1" pin="P"/>
 <pinref part="SW1" gate="G$1" pin="P1"/>
+</segment>
+<segment>
+<pinref part="U1" gate="G$1" pin="!RESETN"/>
+<wire x1="50.324" y1="227.076" x2="44.704" y2="227.076" width="0.1524" layer="91"/>
+<pinref part="R3" gate="G$1" pin="2"/>
+<wire x1="44.704" y1="227.076" x2="44.704" y2="228.156" width="0.1524" layer="91"/>
+<label x="44.196" y="224.79" size="1.778" layer="95"/>
 </segment>
 </net>
@@
 <wire x1="258.216" y1="116.042" x2="276.606" y2="116.042" width="0.1524" layer="91"/>
 </segment>
-</net>
-<net name="N$8" class="0">
 <segment>
 <pinref part="C17" gate="G$1" pin="1"/>
-<wire x1="264.922" y1="116.078" x2="264.842" y2="116.078" width="0.1524" layer="91"/>
-<wire x1="264.842" y1="116.078" x2="264.842" y2="113.91" width="0.1524" layer="91"/>
-<junction x="264.922" y="116.078"/>
-</segment>
-</net>
+<wire x1="264.842" y1="113.91" x2="264.842" y2="116.078" width="0.1524" layer="91"/>
+<wire x1="264.842" y1="116.078" x2="264.668" y2="116.078" width="0.1524" layer="91"/>
+</segment>
+</net>

Commit message: -updated usb pin connections, overlap, ground plane bottom
Connections:
- removed net RST: X1-3.1
- net !RESET: now also X1-3.1
Changed lines of the file:
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@@
 <?xml version="1.0" encoding="utf-8"?>
 <!DOCTYPE eagle SYSTEM "eagle.dtd">
-<eagle version="9.6.1">
+<eagle version="9.5.1">
 <drawing>
 <settings>
-<setting alwaysvectorfont="no"/>
+<setting alwaysvectorfont="yes"/>
 <setting verticaltext="up"/>
 </settings>
@@
 </segment>
 </net>
-<net name="RST" class="0">
-<segment>
-<pinref part="X1" gate="-3" pin="1"/>
-<wire x1="368.554" y1="239.522" x2="371.856" y2="239.522" width="0.1524" layer="91"/>
-<label x="371.856" y="239.522" size="1.778" layer="95" xref="yes"/>
-</segment>
-</net>
 <net name="A0" class="0">
 <segment>
@@
 <label x="44.196" y="224.79" size="1.778" layer="95"/>
 </segment>
-</net>
+<segment>
+<pinref part="X1" gate="-3" pin="1"/>
+<wire x1="368.554" y1="239.522" x2="371.856" y2="239.522" width="0.1524" layer="91"/>
+<label x="371.856" y="239.522" size="1.778" layer="95" xref="yes"/>
+</segment>
+</net>

Commit message: - updated traces - added ring gsm connection
Parts:
- renumbered G1 to RTC-BATT, JP2 to ANT, L to LED13, U1 to SAMDG21, X1 to PROG, X4 to UFL, X6 to RST
Connections:
- removed net D12: SAMDG21.PA19
- removed net RST_D4: SAMDG21.PA08
- new net GSM_RST: SAMDG21.PA19, U$7.RST
- net D4_RST: now also SAMDG21.PA08
Other:
- moved on the sheet: R1, R2
